File: PixelSlasher/PixelSlasher.kicad_pcb (KiCad board)
At the start: 2 copper layers, 52.8 x 149.3 mm, 22 parts, among them J1 VGA Input, J2 CV Red, J3 CV Green, J4 CV Blue, Q1 BC337, Q2 BC337, Q3 BC337, SW1 SW_SPDT, SW2 SW_SPDT, SW3 SW_SPDT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

Commit message: PixelSlasher: 2.1.0: Updated values of R1, R3 and R5 to 51k
Now we're making nearly full use of the slide pots

Signed-off-by: Patrick Pedersen <ctx.xda@gmail.com>
Parts:
- R1, R3, R5: value 40k -> 51k
Connections:
- RV1 pad MP: GND -> (no net)
- RV2 pad MP: GND -> (no net)
- RV3 pad MP: GND -> (no net)
Other:
- board text added: "rev 2.1.0"
- board text removed: "rev 2.0.5"
Changed lines of the file:
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@@
   (title_block
     (date 2019-08-30)
-    (rev 2.0.5)
+    (rev 2.1.0)
     (comment 2 https://www.tapr.org/ohl.html)
     (comment 3 "License: TAPR Open Hardware License v1.0")
@@
   )
   (layers
-    (0 F.Cu signal)
-    (31 B.Cu signal)
+    (0 F.Cu signal hide)
+    (31 B.Cu signal hide)
     (32 B.Adhes user)
     (33 F.Adhes user hide)
@@
     (fp_circle (center 57.25 1.75) (end 58.25 1.75) (layer F.Fab) (width 0.1))
     (fp_circle (center 1.25 1.75) (end 2.25 1.75) (layer F.Fab) (width 0.1))
-    (pad MP thru_hole circle (at 54.35 5.95 90) (size 2.7 2.7) (drill 1.7) (layers *.Cu *.Mask)
-      (net 4 GND))
-    (pad MP thru_hole circle (at 4.15 5.95 90) (size 2.7 2.7) (drill 1.7) (layers *.Cu *.Mask)
-      (net 4 GND))
-    (pad MP thru_hole circle (at 53.15 -2.45 90) (size 2.7 2.7) (drill 1.7) (layers *.Cu *.Mask)
-      (net 4 GND))
-    (pad MP thru_hole circle (at 5.35 -2.45 90) (size 2.7 2.7) (drill 1.7) (layers *.Cu *.Mask)
-      (net 4 GND))
+    (pad MP thru_hole circle (at 54.35 5.95 90) (size 2.7 2.7) (drill 1.7) (layers *.Cu *.Mask))
+    (pad MP thru_hole circle (at 4.15 5.95 90) (size 2.7 2.7) (drill 1.7) (layers *.Cu *.Mask))
+    (pad MP thru_hole circle (at 53.15 -2.45 90) (size 2.7 2.7) (drill 1.7) (layers *.Cu *.Mask))
+    (pad MP thru_hole circle (at 5.35 -2.45 90) (size 2.7 2.7) (drill 1.7) (layers *.Cu *.Mask))
     (pad 3 thru_hole circle (at 58.5 0 90) (size 1.75 1.75) (drill 1.2) (layers *.Cu *.Mask)
       (net 4 GND))
@@
       (effects (font (size 1 1) (thickness 0.15)))
     )
-    (fp_text value BC337 (at -4.346 -0.36) (layer F.Fab)
+    (fp_text value BC337 (at 1.27 -5.09484) (layer F.Fab)
       (effects (font (size 1 1) (thickness 0.15)))
     )
@@
       (effects (font (size 1 1) (thickness 0.15)))
     )
-    (fp_text value 40k (at 3.81 2.37) (layer F.Fab)
+    (fp_text value 51k (at 3.81 2.45) (layer F.Fab)
       (effects (font (size 1 1) (thickness 0.15)))
     )
@@
       (effects (font (size 1 1) (thickness 0.15)))
     )
-    (fp_text value 3.3k (at 3.81 2.37) (layer F.Fab)
+    (fp_text value 3.3k (at 3.81 -2.45) (layer F.Fab)
       (effects (font (size 1 1) (thickness 0.15)))
     )
@@
       (effects (font (size 1 1) (thickness 0.15)))
     )
-    (fp_text value 40k (at 3.81 2.37) (layer F.Fab)
+    (fp_text value 51k (at 3.81 2.45) (layer F.Fab)
       (effects (font (size 1 1) (thickness 0.15)))
     )
@@
       (effects (font (size 1 1) (thickness 0.15)))
     )
-    (fp_text value 3.3k (at 3.81 2.37) (layer F.Fab)
+    (fp_text value 3.3k (at 3.81 2.45) (layer F.Fab)
       (effects (font (size 1 1) (thickness 0.15)))
     )
@@
       (effects (font (size 1 1) (thickness 0.15)))
     )
-    (fp_text value 40k (at 3.81 2.37) (layer F.Fab)
+    (fp_text value 51k (at 3.81 2.45) (layer F.Fab)
       (effects (font (size 1 1) (thickness 0.15)))
     )
@@
       (effects (font (size 1 1) (thickness 0.15)))
     )
-    (fp_text value 3.3k (at 3.81 2.37) (layer F.Fab)
+    (fp_text value 3.3k (at 3.81 2.45) (layer F.Fab)
       (effects (font (size 1 1) (thickness 0.15)))
     )
@@
     (pad 3 thru_hole circle (at 58.5 0 90) (size 1.75 1.75) (drill 1.2) (layers *.Cu *.Mask)
       (net 4 GND))
-    (pad MP thru_hole circle (at 5.35 -2.45 90) (size 2.7 2.7) (drill 1.7) (layers *.Cu *.Mask)
-      (net 4 GND))
-    (pad MP thru_hole circle (at 53.15 -2.45 90) (size 2.7 2.7) (drill 1.7) (layers *.Cu *.Mask)
-      (net 4 GND))
-    (pad MP thru_hole circle (at 4.15 5.95 90) (size 2.7 2.7) (drill 1.7) (layers *.Cu *.Mask)
-      (net 4 GND))
-    (pad MP thru_hole circle (at 54.35 5.95 90) (size 2.7 2.7) (drill 1.7) (layers *.Cu *.Mask)
-      (net 4 GND))
+    (pad MP thru_hole circle (at 5.35 -2.45 90) (size 2.7 2.7) (drill 1.7) (layers *.Cu *.Mask))
+    (pad MP thru_hole circle (at 53.15 -2.45 90) (size 2.7 2.7) (drill 1.7) (layers *.Cu *.Mask))
+    (pad MP thru_hole circle (at 4.15 5.95 90) (size 2.7 2.7) (drill 1.7) (layers *.Cu *.Mask))
+    (pad MP thru_hole circle (at 54.35 5.95 90) (size 2.7 2.7) (drill 1.7) (layers *.Cu *.Mask))
     (model ${KISYS3DMOD}/Potentiometer_THT.3dshapes/Potentiometer_Bourns_PTA4543_Single_Slide.wrl
       (at (xyz 0 0 0))
@@
     (fp_circle (center 57.25 1.75) (end 58.25 1.75) (layer F.Fab) (width 0.1))
     (fp_circle (center 1.25 1.75) (end 2.25 1.75) (layer F.Fab) (width 0.1))
-    (pad MP thru_hole circle (at 54.35 5.95 90) (size 2.7 2.7) (drill 1.7) (layers *.Cu *.Mask)
-      (net 4 GND))
-    (pad MP thru_hole circle (at 4.15 5.95 90) (size 2.7 2.7) (drill 1.7) (layers *.Cu *.Mask)
-      (net 4 GND))
-    (pad MP thru_hole circle (at 53.15 -2.45 90) (size 2.7 2.7) (drill 1.7) (layers *.Cu *.Mask)
-      (net 4 GND))
-    (pad MP thru_hole circle (at 5.35 -2.45 90) (size 2.7 2.7) (drill 1.7) (layers *.Cu *.Mask)
-      (net 4 GND))
+    (pad MP thru_hole circle (at 54.35 5.95 90) (size 2.7 2.7) (drill 1.7) (layers *.Cu *.Mask))
+    (pad MP thru_hole circle (at 4.15 5.95 90) (size 2.7 2.7) (drill 1.7) (layers *.Cu *.Mask))
+    (pad MP thru_hole circle (at 53.15 -2.45 90) (size 2.7 2.7) (drill 1.7) (layers *.Cu *.Mask))
+    (pad MP thru_hole circle (at 5.35 -2.45 90) (size 2.7 2.7) (drill 1.7) (layers *.Cu *.Mask))
     (pad 3 thru_hole circle (at 58.5 0 90) (size 1.75 1.75) (drill 1.2) (layers *.Cu *.Mask)
       (net 4 GND))
@@
       (effects (font (size 1 1) (thickness 0.15)))
     )
-    (fp_text value "CV Red" (at 0 2.33) (layer F.Fab)
+    (fp_text value "CV Red" (at 0 2.74176) (layer F.Fab)
       (effects (font (size 1 1) (thickness 0.15)))
     )
@@
       (effects (font (size 1 1) (thickness 0.15)))
     )
-    (fp_text value "CV Green" (at 0 2.33) (layer F.Fab)
+    (fp_text value "CV Green" (at 0 2.74176) (layer F.Fab)
       (effects (font (size 1 1) (thickness 0.15)))
     )
@@
       (effects (font (size 1 1) (thickness 0.15)))
     )
-    (fp_text value "CV Blue" (at 0 2.33) (layer F.Fab)
+    (fp_text value "CV Blue" (at 0 2.74176) (layer F.Fab)
       (effects (font (size 1 1) (thickness 0.15)))
     )
@@
   (gr_circle (center 111.42 38.5826) (end 112.17 38.5826) (layer Edge.Cuts) (width 0.12))
   (gr_circle (center 149.9108 38.5826) (end 150.6608 38.5826) (layer Edge.Cuts) (width 0.12))
-  (gr_text "rev 2.0.5" (at 130.6068 42.30116) (layer F.SilkS)
+  (gr_text "rev 2.1.0" (at 130.6068 42.30116) (layer F.SilkS)
     (effects (font (size 0.75 0.75) (thickness 0.1)))
   )
